File: tinyK20.sch (KiCad schematic (older format))
At the start: 76 parts, among them CON1 USB-MINI-B, P1 CONN_1, P10 CONN_1, P11 CONN_1, P12 CONN_1, P13 CONN_1, P14 CONN_1, P15 CONN_1, P16 CONN_1, P17 CONN_1, P18 CONN_1, P19 CONN_1, P2 CONN_1, P20 CONN_1, P21 CONN_1, P22 CONN_1, P23 CONN_1, P24 CONN_1, P25 CONN_1, P26 CONN_1, P27 CONN_1, P28 CONN_1, P29 CONN_1, P3 CONN_1, P30 CONN_1, P31 CONN_1, P32 CONN_1, P33 CONN_1, P34 CONN_1, P35 CONN_5X2, P36 CONN_1, P37 CONN_1, P38 CONN_5X2, P4 CONN_1, P40 CONN_1, P5 CONN_1, P6 CONN_1, P7 CONN_1, P8 CONN_1, P9 CONN_1, SW1 SW_PUSH, U1 MK20DX128VFT5, U2 LT1129CST-3.3, U3 74LS126, X1 CRYSTAL_SMD, X2 CRYSTAL_SMD, X3 MOLEX-MICRO-SD

Commit message: k20 schematic
change the sd card socket
Parts:
- removed X1, X2: CRYSTAL_SMD, ~, symbol CRYSTAL_SMD
- removed X3: MOLEX-MICRO-SD, ~, symbol MOLEX-MICRO-SD
- added P34: CONN_1, Connect:PINC, symbol CONN_1
- added P41: CONN_1, Connect:PIN1, symbol CONN_1
- added U4: 105027-0001, symbol 105027-0001
- added Y1: Crystal, Crystals:ABM3, symbol Crystal
- added Y2: Crystal_Small, Crystals:Crystal_Round_Horizontal_3mm_BigPad, symbol Crystal_Small
- C1, C10, C11, C12, C13, C3, C4, C5, C7, C8, C9: footprint ~ -> Capacitors_SMD:C_0805; symbol C -> C-RESCUE-tinyK20
- C2, C6: value 2u2 -> 2.2u; footprint ~ -> Capacitors_SMD:C_0805; symbol C -> C-RESCUE-tinyK20
- CON1: footprint (none) -> Connect:USB_Micro-B
- D1: footprint (none) -> TO_SOT_Packages_SMD:SOT-23
- D2: footprint ~ -> LEDs:LED_0603; symbol LED -> LED-RESCUE-tinyK20
- D3: footprint ~ -> TO_SOT_Packages_SMD:SOT-23
- F1: footprint (none) -> Wire_Connections_Bridges:WireConnection_0.80mmDrill
- GND1: renamed from P12; footprint (none) -> Connect:PIN1
- JP1, JP2, JP3: footprint (none) -> Connect:PINHEAD1-2
- L1, L2, L3: footprint (none) -> Inductors_NEOSID:Neosid_Inductor_SM1206
- P1: renamed from P13; footprint (none) -> Connect:PIN1
- P10: renamed from P22; footprint (none) -> Connect:PIN1
- P11: renamed from P23; footprint (none) -> Connect:PIN1
- P12: renamed from P24; footprint (none) -> Connect:PIN1
- P13: renamed from P25; footprint (none) -> Connect:PIN1
- P14: renamed from P26; footprint (none) -> Connect:PIN1
- P15: renamed from P27; footprint (none) -> Connect:PIN1
- P16: renamed from P28; footprint (none) -> Connect:PIN1
- P17: renamed from P29; footprint (none) -> Connect:PIN1
- P18: renamed from P30; footprint (none) -> Connect:PIN1
- P19: renamed from P31; footprint (none) -> Connect:PIN1
- P2: renamed from P14; footprint (none) -> Connect:PIN1
- P20: renamed from P32; footprint (none) -> Connect:PIN1
- P21: renamed from P33; footprint (none) -> Connect:PIN1
- P22: renamed from P34; footprint (none) -> Connect:PIN1
- P23: renamed from P3; footprint (none) -> Connect:PIN1
- P24: renamed from P37; footprint (none) -> Connect:PINC
- P25: renamed from P5; footprint (none) -> Connect:PINC
- P26: renamed from P6; footprint (none) -> Connect:PINC
- P27: renamed from P8; footprint (none) -> Connect:PIN1
- P28: renamed from P9; footprint (none) -> Connect:PIN1
- P29: renamed from P11; footprint (none) -> Connect:PIN1
- P3: renamed from P15; footprint (none) -> Connect:PIN1
- P30: renamed from P10; footprint (none) -> Connect:PIN1
- P31: renamed from P7; footprint (none) -> Connect:PIN1
- P32: renamed from P4; footprint (none) -> Connect:PINC
- P33: renamed from P1; footprint (none) -> Connect:PIN1
- P35, P38: footprint (none) -> Pin_Headers:Pin_Header_Straight_2x05_Pitch1.27mm
- P36: renamed from P2; footprint (none) -> Connect:PINC
- P37: renamed from P36; footprint (none) -> Connect:PINC
- P4: renamed from P16; footprint (none) -> Connect:PIN1
- P5: renamed from P17; footprint (none) -> Connect:PIN1
- P6: renamed from P18; footprint (none) -> Connect:PIN1
- P7: renamed from P19; footprint (none) -> Connect:PIN1
- P8: renamed from P20; footprint (none) -> Connect:PIN1
- P9: renamed from P21; footprint (none) -> Connect:PIN1
- R1, R2, R3, R5: footprint ~ -> Resistors_SMD:R_0805; symbol R -> R-RESCUE-tinyK20
- R4, R6: value R -> 1k; footprint ~ -> Resistors_SMD:R_0805; symbol R -> R-RESCUE-tinyK20
- SW1: footprint ~ -> Buttons_Switches_SMD:SW_SPST_EVQPE1
- U1: footprint ~ -> Housings_DFN_QFN:QFN-48-1EP_7x7mm_Pitch0.5mm; symbol MK20DX128VFT5 -> MK20DX128VFT5-RESCUE-tinyK20
- U2: footprint SOT-223 -> TO_SOT_Packages_SMD:SOT-223
- U3: footprint ~ -> SMD_Packages:SOIC-14_N
- VBATT1: renamed from P40; footprint (none) -> Connect:PIN1
Connections:
- net labels added: Vreg, x+, x-, xtal_N, xtal_P
- net labels removed: 5V, UART_RX, UART_TX
- wire segments 231 -> 234
Other:
- note added: "USB port"
- moved on the sheet: C1, C10, C11, C12, C13, C2, C3, C4, C5, C6, C7, C8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

Commit message: Add files via upload
add two 22nF capacitors and a 33M resistor to the crystal Y1
Parts:
- added C14, C15: 22nF, Capacitors_SMD:C_0805, symbol C
- added R7: 1M, Capacitors_SMD:C_0402, symbol R
- P35, P38: footprint Pin_Headers:Pin_Header_Straight_2x05_Pitch1.27mm -> Connect:CONN-2x5-1.27-SMT
Connections:
- wire segments 234 -> 243
Changed lines of the file:
@@
 $EndComp
 $Comp
-L GND-RESCUE-tinyK20 #PWR1
+L GND-RESCUE-tinyK20 #PWR01
 U 1 1 56D0B4EA
 P 1175 5850
-F 0 "#PWR1" H 1175 5850 30  0001 C CNN
+F 0 "#PWR01" H 1175 5850 30  0001 C CNN
 F 1 "GND" H 1175 5780 30  0001 C CNN
 F 2 "" H 1175 5850 60  0000 C CNN
@@
 $EndComp
 $Comp
-L GND-RESCUE-tinyK20 #PWR16
+L GND-RESCUE-tinyK20 #PWR02
 U 1 1 56D0C4E9
 P 6850 3050
-F 0 "#PWR16" H 6850 3050 30  0001 C CNN
+F 0 "#PWR02" H 6850 3050 30  0001 C CNN
 F 1 "GND" H 6850 2980 30  0001 C CNN
 F 2 "" H 6850 3050 60  0000 C CNN
@@
 $EndComp
 $Comp
-L GND-RESCUE-tinyK20 #PWR14
+L GND-RESCUE-tinyK20 #PWR03
 U 1 1 56D158C9
 P 5350 6025
-F 0 "#PWR14" H 5350 6025 30  0001 C CNN
+F 0 "#PWR03" H 5350 6025 30  0001 C CNN
 F 1 "GND" H 5350 5955 30  0001 C CNN
 F 2 "" H 5350 6025 60  0000 C CNN
@@
 $EndComp
 $Comp
-L 3V3 #PWR13
+L 3V3 #PWR04
 U 1 1 56D15AFA
 P 5350 5375
-F 0 "#PWR13" H 5350 5475 40  0001 C CNN
+F 0 "#PWR04" H 5350 5475 40  0001 C CNN
 F 1 "3V3" H 5350 5500 40  0000 C CNN
 F 2 "" H 5350 5375 60  0000 C CNN
@@
 $EndComp
 $Comp
-L 3V3 #PWR17
+L 3V3 #PWR05
 U 1 1 56D15B9F
 P 8050 2400
-F 0 "#PWR17" H 8050 2500 40  0001 C CNN
+F 0 "#PWR05" H 8050 2500 40  0001 C CNN
 F 1 "3V3" H 8050 2525 40  0000 C CNN
 F 2 "" H 8050 2400 60  0000 C CNN
@@
 $EndComp
 $Comp
-L GND-RESCUE-tinyK20 #PWR15
+L GND-RESCUE-tinyK20 #PWR06
 U 1 1 56D173DE
 P 6300 9050
-F 0 "#PWR15" H 6300 9050 30  0001 C CNN
+F 0 "#PWR06" H 6300 9050 30  0001 C CNN
 F 1 "GND" H 6300 8980 30  0001 C CNN
 F 2 "" H 6300 9050 60  0000 C CNN
@@
 D+
 $Comp
-L PWR_FLAG #FLG2
+L PWR_FLAG #FLG07
 U 1 1 56D1AD9A
 P 6950 2400
-F 0 "#FLG2" H 6950 2495 30  0001 C CNN
+F 0 "#FLG07" H 6950 2495 30  0001 C CNN
 F 1 "PWR_FLAG" H 6950 2580 30  0000 C CNN
 F 2 "" H 6950 2400 60  0000 C CNN
@@
 $EndComp
 $Comp
-L 3V3 #PWR20
+L 3V3 #PWR08
 U 1 1 56D1AF46
 P 12475 5800
-F 0 "#PWR20" H 12475 5900 40  0001 C CNN
+F 0 "#PWR08" H 12475 5900 40  0001 C CNN
 F 1 "3V3" H 12475 5925 40  0000 C CNN
 F 2 "" H 12475 5800 60  0000 C CNN
@@
 $EndComp
 $Comp
-L PWR_FLAG #FLG3
+L PWR_FLAG #FLG09
 U 1 1 56D1B8A7
 P 7500 3075
-F 0 "#FLG3" H 7500 3170 30  0001 C CNN
+F 0 "#FLG09" H 7500 3170 30  0001 C CNN
 F 1 "PWR_FLAG" H 7500 3255 30  0000 C CNN
 F 2 "" H 7500 3075 60  0000 C CNN
@@
 $EndComp
 $Comp
-L GND-RESCUE-tinyK20 #PWR12
+L GND-RESCUE-tinyK20 #PWR010
 U 1 1 56D1BB5D
 P 4825 7475
-F 0 "#PWR12" H 4825 7475 30  0001 C CNN
+F 0 "#PWR010" H 4825 7475 30  0001 C CNN
 F 1 "GND" H 4825 7405 30  0001 C CNN
 F 2 "" H 4825 7475 60  0000 C CNN
@@
 $EndComp
 $Comp
-L 3V3 #PWR11
+L 3V3 #PWR011
 U 1 1 56D1BC38
 P 4175 6850
-F 0 "#PWR11" H 4175 6950 40  0001 C CNN
+F 0 "#PWR011" H 4175 6950 40  0001 C CNN
 F 1 "3V3" H 4175 6975 40  0000 C CNN
 F 2 "" H 4175 6850 60  0000 C CNN
@@
 $EndComp
 $Comp
-L GND-RESCUE-tinyK20 #PWR7
+L GND-RESCUE-tinyK20 #PWR012
 U 1 1 56D1BFC1
 P 3175 6650
-F 0 "#PWR7" H 3175 6650 30  0001 C CNN
+F 0 "#PWR012" H 3175 6650 30  0001 C CNN
 F 1 "GND" H 3175 6580 30  0001 C CNN
 F 2 "" H 3175 6650 60  0000 C CNN
@@
 F 0 "P35" H 2400 2525 60  0000 C CNN
 F 1 "CONN_5X2" V 2400 2225 50  0000 C CNN
-F 2 "Pin_Headers:Pin_Header_Straight_2x05_Pitch1.27mm" H 2400 2225 60  0001 C CNN
+F 2 "Connect:CONN-2x5-1.27-SMT" H 2400 2225 60  0001 C CNN
 F 3 "" H 2400 2225 60  0000 C CNN
 	1    2400 2225
@@
 $EndComp
 $Comp
-L 3V3 #PWR4
+L 3V3 #PWR013
 U 1 1 56D1C1ED
 P 1925 1800
-F 0 "#PWR4" H 1925 1900 40  0001 C CNN
+F 0 "#PWR013" H 1925 1900 40  0001 C CNN
 F 1 "3V3" H 1925 1925 40  0000 C CNN
 F 2 "" H 1925 1800 60  0000 C CNN
@@
 $EndComp
 $Comp
-L GND-RESCUE-tinyK20 #PWR3
+L GND-RESCUE-tinyK20 #PWR014
 U 1 1 56D1C1FC
 P 1800 2575
-F 0 "#PWR3" H 1800 2575 30  0001 C CNN
+F 0 "#PWR014" H 1800 2575 30  0001 C CNN
 F 1 "GND" H 1800 2505 30  0001 C CNN
 F 2 "" H 1800 2575 60  0000 C CNN
@@
 $EndComp
 $Comp
-L GND-RESCUE-tinyK20 #PWR9
+L GND-RESCUE-tinyK20 #PWR015
 U 1 1 56D1C496
 P 3675 3275
-F 0 "#PWR9" H 3675 3275 30  0001 C CNN
+F 0 "#PWR015" H 3675 3275 30  0001 C CNN
 F 1 "GND" H 3675 3205 30  0001 C CNN
 F 2 "" H 3675 3275 60  0000 C CNN
@@
 $EndComp
 $Comp
-L GND-RESCUE-tinyK20 #PWR10
+L GND-RESCUE-tinyK20 #PWR016
 U 1 1 56D1C4A5
 P 3975 3275
-F 0 "#PWR10" H 3975 3275 30  0001 C CNN
+F 0 "#PWR016" H 3975 3275 30  0001 C CNN
 F 1 "GND" H 3975 3205 30  0001 C CNN
 F 2 "" H 3975 3275 60  0000 C CNN
@@
 UART1_TX
 $Comp
-L 3V3 #PWR8
+L 3V3 #PWR017
 U 1 1 56D1CB0F
 P 3675 1825
-F 0 "#PWR8" H 3675 1925 40  0001 C CNN
+F 0 "#PWR017" H 3675 1925 40  0001 C CNN
 F 1 "3V3" H 3675 1950 40  0000 C CNN
 F 2 "" H 3675 1825 60  0000 C CNN
@@
 Target SWD interface
 $Comp
-L +3.3V-RESCUE-tinyK20 #PWR6
+L +3.3V-RESCUE-tinyK20 #PWR018
 U 1 1 56D4C67E
 P 2025 8525
-F 0 "#PWR6" H 2025 8485 30  0001 C CNN
+F 0 "#PWR018" H 2025 8485 30  0001 C CNN
 F 1 "+3.3V" H 2025 8635 30  0000 C CNN
 F 2 "" H 2025 8525 60  0000 C CNN
@@
 $EndComp
 $Comp
-L GND-RESCUE-tinyK20 #PWR2
+L GND-RESCUE-tinyK20 #PWR019
 U 1 1 56D4C6A1
 P 1725 9175
-F 0 "#PWR2" H 1725 9175 30  0001 C CNN
+F 0 "#PWR019" H 1725 9175 30  0001 C CNN
 F 1 "GND" H 1725 9105 30  0001 C CNN
 F 2 "" H 1725 9175 60  0000 C CNN
@@
 PTC1
 $Comp
-L GND-RESCUE-tinyK20 #PWR5
+L GND-RESCUE-tinyK20 #PWR020
 U 1 1 56D4DD26
 P 1975 10400
-F 0 "#PWR5" H 1975 10400 30  0001 C CNN
+F 0 "#PWR020" H 1975 10400 30  0001 C CNN
 F 1 "GND" H 1975 10330 30  0001 C CNN
 F 2 "" H 1975 10400 60  0000 C CNN
@@
 PTC0
 $Comp
-L PWR_FLAG #FLG1
+L PWR_FLAG #FLG021
 U 1 1 56D50D28
 P 2200 8625
-F 0 "#FLG1" H 2200 8720 30  0001 C CNN
+F 0 "#FLG021" H 2200 8720 30  0001 C CNN
 F 1 "PWR_FLAG" H 2200 8805 30  0000 C CNN
 F 2 "" H 2200 8625 60  0000 C CNN
@@
 F 0 "P38" H 12250 3275 60  0000 C CNN
 F 1 "CONN_5X2" V 12250 2975 50  0000 C CNN
-F 2 "Pin_Headers:Pin_Header_Straight_2x05_Pitch1.27mm" H 12250 2975 60  0001 C CNN
+F 2 "Connect:CONN-2x5-1.27-SMT" H 12250 2975 60  0001 C CNN
 F 3 "" H 12250 2975 60  0000 C CNN
 	1    12250 2975
@@
 PTB1
 $Comp
-L GND-RESCUE-tinyK20 #PWR18
+L GND-RESCUE-tinyK20 #PWR022
 U 1 1 56D51882
 P 9875 3350
-F 0 "#PWR18" H 9875 3350 30  0001 C CNN
+F 0 "#PWR022" H 9875 3350 30  0001 C CNN
 F 1 "GND" H 9875 3280 30  0001 C CNN
 F 2 "" H 9875 3350 60  0000 C CNN
@@
 $EndComp
 $Comp
-L 3V3 #PWR19
+L 3V3 #PWR023
 U 1 1 56D518AF
 P 10025 2775
-F 0 "#PWR19" H 10025 2875 40  0001 C CNN
+F 0 "#PWR023" H 10025 2875 40  0001 C CNN
 F 1 "3V3" V 10025 2975 40  0000 C CNN
 F 2 "" H 10025 2775 60  0000 C CNN
@@
 $EndComp
 $Comp
-L PWR_FLAG #FLG4
+L PWR_FLAG #FLG024
 U 1 1 56D534BA
 P 10675 2325
-F 0 "#FLG4" H 10675 2420 30  0001 C CNN
+F 0 "#FLG024" H 10675 2420 30  0001 C CNN
 F 1 "PWR_FLAG" H 10675 2505 30  0000 C CNN
 F 2 "" H 10675 2325 60  0000 C CNN
@@
 	0    1    1    0
 $EndComp
+$Comp
+L R R7
+U 1 1 5738953E
+P 5275 9150
+F 0 "R7" V 5355 9150 50  0000 C CNN
+F 1 "1M" V 5275 9150 50  0000 C CNN
+F 2 "Capacitors_SMD:C_0402" V 5205 9150 50  0001 C CNN
+F 3 "" H 5275 9150 50  0000 C CNN
+	1    5275 9150
+	0    1    1    0
+$EndComp
+$Comp
+L C C14
+U 1 1 5739AF46
+P 5250 8825
+F 0 "C14" H 5275 8925 50  0000 L CNN
+F 1 "22nF" H 5275 8725 50  0000 L CNN
+F 2 "Capacitors_SMD:C_0805" H 5288 8675 50  0001 C CNN
+F 3 "" H 5250 8825 50  0000 C CNN
+	1    5250 8825
+	0    1    1    0
+$EndComp
 Wire Wire Line
 	6050 2050 6050 2350
@@
 	5750 8525 5875 8525
 Wire Wire Line
-	5875 8525 5875 8425
+	5875 8425 5875 8750
 Wire Wire Line
 	5875 8425 6350 8425
@@
 	6225 5525 6350 5525
 Wire Wire Line
-	5400 8525 5450 8525
-Wire Wire Line
 	6125 6875 6350 6875
 Wire Wire Line
@@
 Wire Wire Line
 	1475 9300 2025 9300
+Connection ~ 5400 8525
+Wire Wire Line
+	4875 9150 5125 9150
+Wire Wire Line
+	4875 8525 4875 9150
+Wire Wire Line
+	4875 8825 5100 8825
+Wire Wire Line
+	5450 8525 4875 8525
+Connection ~ 4875 8825
+Wire Wire Line
+	5400 8825 6225 8825
+Wire Wire Line
+	6225 8825 6225 9150
+Connection ~ 6225 8875
+$Comp
+L C C15
+U 1 1 573A6F5F
+P 5775 9150
+F 0 "C15" H 5800 9250 50  0000 L CNN
+F 1 "22nF" H 5800 9050 50  0000 L CNN
+F 2 "Capacitors_SMD:C_0805" H 5813 9000 50  0001 C CNN
+F 3 "" H 5775 9150 50  0000 C CNN
+	1    5775 9150
+	0    1    1    0
+$EndComp
+Wire Wire Line
+	5425 9150 5625 9150
+Wire Wire Line
+	5875 8750 5550 8750
+Wire Wire Line
+	5550 8750 5550 9150
+Connection ~ 5550 9150
+Connection ~ 5875 8525
+Wire Wire Line
+	6225 9150 5925 9150
 $EndSCHEMATC
