File: tinyK20.sch (KiCad schematic (older format))
At the start: 79 parts, among them CON1 USB-MINI-B, P1 CONN_1, P10 CONN_1, P11 CONN_1, P12 CONN_1, P13 CONN_1, P14 CONN_1, P15 CONN_1, P16 CONN_1, P17 CONN_1, P18 CONN_1, P19 CONN_1, P2 CONN_1, P20 CONN_1, P21 CONN_1, P22 CONN_1, P23 CONN_1, P24 CONN_1, P25 CONN_1, P26 CONN_1, P27 CONN_1, P28 CONN_1, P29 CONN_1, P3 CONN_1, P30 CONN_1, P31 CONN_1, P33 CONN_1, P34 CONN_1, P35 CONN_5X2, P37 CONN_1, P38 CONN_5X2, P4 CONN_1, P41 CONN_1, P5 CONN_1, P6 CONN_1, P7 CONN_1, P8 CONN_1, P9 CONN_1, SW1 SW_PUSH, U1 MK20DX128VFT5, U2 LT1129CST-3.3, U3 74LS126, U4 105027-0001, Y1 Crystal, Y2 Crystal_Small

Commit message: Get rid of ground plane on top copper.
 Add optional vias. Re-route tracks
Parts:
- removed C12: 2.2u, Capacitors_SMD:C_0805, symbol C-RESCUE-tinyK20
- removed GND1, P1, P10, P11, P12, P13, P14, P15, P16, P17, P18, P19, P2, P20, P21, P22, P23, P27, P28, P29, P3, P30, P31, P33, P4, P41, P5, P6, P7, P8, P9: CONN_1, Connect:PIN1, symbol CONN_1
- removed P24, P25, P26, P34, P37: CONN_1, Connect:PINC, symbol CONN_1
- removed U4: 105027-0001, symbol 105027-0001
- D2: footprint LEDs:LED_0603 -> Resistors_SMD:R_1206
- P35: footprint Connect:CONN-2x5-1.27-SMT -> Pin_Headers:Pin_Header_Straight_2x05_Pitch1.27mm
- R1, R4, R6: footprint Resistors_SMD:R_0805 -> Resistors_SMD:R_1206_HandSoldering
- R2, R3: footprint Resistors_SMD:R_0805 -> Resistors_SMD:R_0603_HandSoldering
- R5: footprint Resistors_SMD:R_0805 -> Resistors_SMD:R_1206
- R7: footprint Capacitors_SMD:C_0402 -> Resistors_SMD:R_1206_HandSoldering
- VBATT1: footprint Connect:PIN1 -> Wire_Pads:SolderWirePad_single_1mmDrill
- Y1: footprint Crystals:ABM3 -> Housings_DFN_QFN:ABM3
Connections:
- net labels removed: PTC0, PTC1
- wire segments 239 -> 180
- no-connect marks 6 -> 23
Other:
- note removed: "opt. micro-SD card interface"
- moved on the sheet: JP2, JP3
